File: pn5180 cat5 connector with linear regulator/pn5180 cat5 connector with linear regulator.kicad_sch (KiCad schematic)
At the start: 5 parts, among them J1 RJ45_Shielded, J2 Conn_01x09_Pin, U1 AMS1117-3.3

Commit message: asdf
Parts:
- C1, C2: value C -> 10uF
Changed lines of the file:
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@@
       (effects (font (size 1.27 1.27)) (justify left))
     )
-    (property "Value" "C" (at 148.59 120.015 0)
+    (property "Value" "10uF" (at 148.59 120.015 0)
       (effects (font (size 1.27 1.27)) (justify left))
     )
@@
       (effects (font (size 1.27 1.27)) (justify left))
     )
-    (property "Value" "C" (at 133.35 120.015 0)
+    (property "Value" "10uF" (at 133.35 120.015 0)
       (effects (font (size 1.27 1.27)) (justify left))
     )
