File: pn5180 cat5 connector with linear regulator/pn5180 cat5 connector with linear regulator.kicad_pcb (KiCad board)
At the start: 2 copper layers, 25.4 x 24.4 mm, 5 parts, among them J1 RJ45_Shielded, J2 Conn_01x09_Pin, U1 AMS1117-3.3

Commit message: Update pn5180 cat5 connector with linear regulator.kicad_pcb
Parts:
- C1, C2: value C -> 10uF
Changed lines of the file:
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@@
         (effects (font (size 1 1) (thickness 0.15)))
     )
-    (fp_text value "C" (at 2.5 2.5) (layer "F.Fab")
+    (fp_text value "10uF" (at 2.445 -2.967) (layer "F.Fab")
         (effects (font (size 1 1) (thickness 0.15)))
     )
@@
         (effects (font (size 1 1) (thickness 0.15)))
     )
-    (fp_text value "C" (at 2.5 2.5) (layer "F.Fab")
+    (fp_text value "10uF" (at 2.5 2.5) (layer "F.Fab")
         (effects (font (size 1 1) (thickness 0.15)))
     )
