File: Shift Register Mosfet Array V3/Shift Register Mosfet Array V3.kicad_pcb (KiCad board)
At the start: 2 copper layers, 97.5 x 53.9 mm, 77 parts, among them J1 Conn_01x06_Pin, J10 Conn_01x01_Pin, J11 Conn_01x02_Pin, J12 Conn_01x01_Pin, J13 Conn_01x02_Pin, J14 Conn_01x01_Pin, J15 Conn_01x02_Pin, J16 Conn_01x01_Pin, J17 Conn_01x02_Pin, J18 Conn_01x06_Pin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

Commit message: Update Shift Register Mosfet Array V3.kicad_pcb
Parts:
- moved D2 2.34 mm to (75.3, 139.2)
- moved D3 2.34 mm to (85.1, 139.2)
- moved D4 2.34 mm to (95.3, 139.2)
- moved D5 2.34 mm to (105.2, 139.2)
- moved D6 2.34 mm to (115.4, 139.2)
- moved D7 2.34 mm to (125.3, 139.2)
- moved D8 2.34 mm to (135.2, 139.2)
- moved D9 2.34 mm to (145.3, 139.2)
- moved J10 2.34 mm to (128.8, 132.3)
- moved J11 2.34 mm to (116.3, 132.3)
- moved J12 2.34 mm to (138.8, 132.3)
- moved J13 2.34 mm to (126.3, 132.3)
- moved J14 2.34 mm to (78.8, 132.3)
- moved J15 2.34 mm to (136.3, 132.3)
- moved J16 2.34 mm to (148.8, 132.3)
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Routing:
- net 12V: track 209.0 -> 215.1 mm
- net Net-(D11-A): track 19.9 -> 22.2 mm
- net Net-(D17-A): track 22.8 -> 25.1 mm
- net Net-(D16-A): track 19.9 -> 22.2 mm
- net Net-(D15-A): track 19.0 -> 21.4 mm
- net Net-(D14-A): track 26.5 -> 28.8 mm
- net Net-(D13-A): track 21.1 -> 23.5 mm
- net Net-(D12-A): track 19.6 -> 22.0 mm
- net Net-(D10-A): track 22.0 -> 24.3 mm
